File: portabeer_pcb/portabeer_pcb.kicad_pcb (KiCad board)
At the start: 2 copper layers, 100 x 100 mm, 285 parts, among them J1 USB_B_Micro, J10 Conn_01x03, J11 Conn_01x03, J12 Conn_01x03, J13 XT60IPW, J14 Barrel_Jack_MountingPin, J15 Conn_01x03, J16 Conn_01x03, J17 Conn_01x03, J18 Conn_01x03, J2 GMG12864-06D, J3 Conn_01x03, J4 I2C expansion, J5 Conn_01x03, J6 Conn_01x03, J7 Conn_01x03, J8 Conn_01x03, J9 Conn_01x03, M1 Air pump, M3 Water pump, M4 Air pump, M6 Water pump, M7 Fan_4pin, M8 Fan_4pin, Q1 AO3400A, Q10 AO3400A, Q11 AO3400A, Q12 Si7336ADP, Q13 Si7336ADP, Q16 Si7336ADP, Q17 Si7336ADP, Q2 BSS84, Q3 BSS138, Q4 Si7145DP, Q5 Si7145DP, Q6 SiS454DN, Q7 AO3400A, Q8 AO3400A, Q9 SiS454DN, SW1 RESET, SW2 BOOTSEL, SW3 RotaryEncoder_Switch_MP, U1 USBLC6-2SC6, U10 LTC4412xS6, U11 MP26124, U12 GBI7254MMAR, U14 TPS92640PWP/NOPB, U15 TPS92640PWP/NOPB, U16 MCP47FEB12, U18 REF3025, U2 W25Q128JVS, U3 RP2040, U4 PCA9536DP, U5 XC6206PxxxMR, U6 TPS54202DDC, U7 LTC2954-1, U8 ADS7828, U9 LTC2943, Y1 Crystal_GND24

Commit message: electronics diagram and schematic
Parts:
- added BZ1: Buzzer, Buzzer_Beeper:MagneticBuzzer_CUI_CST-931RP-A, F.Cu at (178.2, 101.0)
- added C20: C_Polarized, Capacitor_THT:CP_Radial_D6.3mm_P2.50mm, F.Cu at (143.8, 123.2)
- added C22: C_Polarized, Capacitor_THT:CP_Radial_D6.3mm_P2.50mm, F.Cu at (157.2, 78.0)
- added C27: C_Polarized, Capacitor_THT:CP_Radial_D6.3mm_P2.50mm, F.Cu at (158.1, 99.2)
- added C54: C_Polarized, Capacitor_THT:CP_Radial_D6.3mm_P2.50mm, F.Cu at (-55.8, 61.4)
- added C57: C_Polarized, Capacitor_THT:CP_Radial_D8.0mm_P3.50mm, F.Cu at (-47.7, 63.0)
- added C60: C_Polarized, Capacitor_THT:CP_Radial_D6.3mm_P2.50mm, F.Cu at (-55.8, 69.2)
- added C66: C_Polarized, Capacitor_THT:CP_Radial_D10.0mm_P5.00mm, F.Cu at (248.0, 87.2)
- added C67: C_Polarized, Capacitor_THT:CP_Radial_D8.0mm_P3.50mm, F.Cu at (73.6, 181.2)
- added C71: C_Polarized, Capacitor_THT:CP_Radial_D10.0mm_P5.00mm, F.Cu at (109.4, -78.2)
- added C73: C_Polarized, Capacitor_THT:CP_Radial_D6.3mm_P2.50mm, F.Cu at (83.5, 178.8)
- added C74: C_Polarized, Capacitor_THT:CP_Radial_D6.3mm_P2.50mm, F.Cu at (91.2, 182.2)
- added C82: C_Polarized, Capacitor_THT:CP_Radial_D8.0mm_P3.50mm, F.Cu at (161.3, -49.0)
- added C88: C_Polarized, Capacitor_THT:CP_Radial_D6.3mm_P2.50mm, F.Cu at (161.5, -27.8)
- added C89: C_Polarized, Capacitor_THT:CP_Radial_D6.3mm_P2.50mm, F.Cu at (162.3, -17.5)
- added Q14: AO3400A, Package_TO_SOT_SMD:SOT-23, F.Cu at (158.8, 53.6)
- added R51: 10k, Resistor_SMD:R_0603_1608Metric, F.Cu at (158.4, 47.4)
- added R52: 10, Resistor_SMD:R_0603_1608Metric, F.Cu at (158.4, 49.9)
- added R53: R, Resistor_SMD:R_0805_2012Metric, F.Cu at (158.6, 57.2)
- D15, D16: footprint Diode_SMD:D_SOD-523 -> Diode_SMD:D_SOD-123
- Q3: footprint Package_TO_SOT_SMD:SOT-523 -> Package_TO_SOT_SMD:SOT-23
- R42: value 100K -> 470k
- R45: value 10k -> 470k
- moved C1 341.8 mm to (215.0, 75.5)
- moved C2 341.8 mm to (215.0, 83.0)
- moved R2 341.8 mm to (215.0, 77.0)
- moved R3 341.8 mm to (215.0, 81.5)
- moved R5 341.8 mm to (215.0, 78.5)
- moved R6 341.8 mm to (215.0, 80.0)
- moved SW3 341.8 mm to (218.0, 76.8)
- moved R89 40.0 mm to (267.2, 98.8), turned to 0 degrees
- moved R87 38.4 mm to (263.0, 99.5), turned to 180 degrees
- moved R90 38.1 mm to (267.2, 97.2), turned to 0 degrees
- moved R88 37.1 mm to (260.0, 99.5), turned to 180 degrees
- moved C98 36.3 mm to (267.2, 95.8), turned to 0 degrees
- moved C95 36.0 mm to (255.8, 99.5), turned to 180 degrees
- moved D15 34.6 mm to (267.2, 94.2), turned to 0 degrees
- moved C78 33.9 mm to (255.8, 98.0), turned to 180 degrees
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Connections:
- R15 pad 2: /MCU/GPIO25 -> +3.3V
- U3 pad 37: /MCU/GPIO25 -> /MCU/BUZZ
Routing:
- net /FAN_TACH_1: track 1.79 -> 10.1 mm
- net /MCU/DAC_REF: track 0.00 -> 5.66 mm
- net +BATT: track 0.00 -> 4.55 mm
- net /Battery/BATT_P: track 0.00 -> 3.95 mm
- net Net-(U16-~{LAT}/HVC): track 0.00 -> 3.72 mm
- net /FAN_EN_1: track 0.00 -> 3.31 mm
- net +3.3V: track 89.6 -> 92.7 mm
- net /WP_EN_1: track 0.00 -> 3.05 mm
- net Net-(Q8-G): track 0.00 -> 1.92 mm
- net Net-(Q7-G): track 0.00 -> 1.92 mm
- net /SDA: track 0.00 -> 1.40 mm
- net /SCL: track 0.00 -> 1.40 mm
- added copper zone on F.Cu, net /Dispenser 1/FAN
- added copper zone on F.Cu, net /Dispenser 1/WP

Commit message: added 3d models, started layout
Parts:
- removed C54, C60, C73, C74, C88, C89: C_Polarized, Capacitor_THT:CP_Radial_D6.3mm_P2.50mm
- removed C67, C82: C_Polarized, Capacitor_THT:CP_Radial_D8.0mm_P3.50mm
- removed C68, C81: 10u, Capacitor_SMD:C_1206_3216Metric
- removed R75: 100, Resistor_SMD:R_0603_1608Metric
- removed R99: 1k, Resistor_SMD:R_0603_1608Metric
- removed U18: REF3025, Package_TO_SOT_SMD:SOT-23
- removed U4: PCA9536DP, Package_SO:TSSOP-8_3x3mm_P0.65mm
- added R54: 100, Resistor_SMD:R_0603_1608Metric, F.Cu at (232.7, 47.2)
- added R59: 1k, Resistor_SMD:R_0603_1608Metric, F.Cu at (218.2, 89.0)
- added U13: GBI7254MMAR, Package_SO:MSOP-8-1EP_3x3mm_P0.65mm_EP1.95x2.15mm, F.Cu at (254.0, 104.2)
- added U17: REF3012, Package_TO_SOT_SMD:SOT-23, F.Cu at (222.2, 95.4)
- BZ1, J2: moved to B.Cu
- C66, C71: footprint Capacitor_THT:CP_Radial_D10.0mm_P5.00mm -> Capacitor_THT:CP_Radial_D8.0mm_P3.50mm
- J1: footprint Connector_USB:USB_Micro-B_Amphenol_10118193-0001LF_Horizontal -> portabeer:USB_Micro-B_Amphenol_10118193-0001LF_Horizontal
- J13: footprint Connector_AMASS:AMASS_XT60IPW-M_1x03_P7.20mm_Horizontal -> portabeer:AMASS_XT60IPW-M_1x03_P7.20mm_Horizontal
- L1: footprint Inductor_SMD:L_Taiyo-Yuden_NR-40xx -> portabeer:L_Taiyo-Yuden_NR-40xx
- L2: footprint Inductor_SMD:L_Taiyo-Yuden_NR-50xx -> portabeer:L_Taiyo-Yuden_NR-50xx
- Q12, Q13, Q16, Q17, Q4, Q5: footprint Package_SO:PowerPAK_SO-8_Single -> portabeer:PowerPAK_SO-8_Single
- Q6, Q9: footprint Package_SO:Vishay_PowerPAK_1212-8_Single -> portabeer:Vishay_PowerPAK_1212-8_Single
- R2: value 10Rx -> 10k
- R3: value 10Rx -> 10
- R41: value R -> 3m
- R5, R6: value Rx -> 10Rx
- R51: value 10k -> 10
- R52: value 10 -> 10k
- R8: value 10k -> Rx
- R9: value 10 -> Rx
- SW3: footprint Rotary_Encoder:RotaryEncoder_Alps_EC11E-Switch_Vertical_H20mm -> portabeer:RotaryEncoder_Alps_EC11E-Switch_Vertical_H20mm; moved to B.Cu
- U12: value GBI7254MMAR -> PCA9536DP; footprint Package_SO:MSOP-8-1EP_3x3mm_P0.65mm_EP1.95x2.15mm -> Package_SO:TSSOP-8_3x3mm_P0.65mm
- U2: footprint Package_SO:SOIC-8_5.23x5.23mm_P1.27mm -> portabeer:SOIC-8_5.23x5.23mm_P1.27mm
- U9: footprint Package_DFN_QFN:DFN-8-1EP_3x3mm_P0.5mm_EP1.65x2.38mm -> portabeer:DFN-8-1EP_3x3mm_P0.5mm_EP1.65x2.38mm
- moved C57 323.7 mm to (272.7, 109.5), turned to 180 degrees
- moved C83 287.1 mm to (238.3, 44.2)
- moved C108 282.5 mm to (232.7, 44.7), turned to 0 degrees
- moved J12 278.9 mm to (273.2, 39.3), turned to 180 degrees
- moved J11 274.2 mm to (273.2, 44.0), turned to 180 degrees
- moved J10 269.8 mm to (273.2, 48.8), turned to 180 degrees
- moved R32 267.3 mm to (266.0, 38.5), turned to 90 degrees
- moved J9 265.7 mm to (273.2, 53.5), turned to 180 degrees
- moved C42 264.7 mm to (264.5, 38.5), turned to -90 degrees
- moved R31 262.4 mm to (266.0, 43.2), turned to 90 degrees
- moved J8 261.9 mm to (273.2, 58.3), turned to 180 degrees
- moved C41 259.8 mm to (264.5, 43.2), turned to -90 degrees
- moved C86 259.4 mm to (222.0, 96.6), turned to 0 degrees
- moved J7 258.3 mm to (273.2, 63.0), turned to 180 degrees
- moved U16 258.1 mm to (217.5, 93.8), turned to 90 degrees
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Connections:
- net /Battery/BATT_P renamed /BAT/BATT_PF
- net /Battery/CHG_CS+ renamed /BAT/CHG_CS+
- net /Battery/CHG_CS- renamed /BAT/CHG_CS-
- net /Battery/CHG_SW renamed /BAT/CHG_SW
- net /Battery/CHG_VREF renamed /BAT/CHG_VREF
- net /Battery/STAT renamed /BAT/STAT
- net /Dispenser 1/AP renamed /KEG1/AP
- net /Dispenser 1/Driver/BOOT renamed /KEG1/Driver/BOOT
- net /Dispenser 1/Driver/CS renamed /KEG1/Driver/CS
- net /Dispenser 1/Driver/HG renamed /KEG1/Driver/HG
- net /Dispenser 1/Driver/LG renamed /KEG1/Driver/LG
- net /Dispenser 1/Driver/OUT+ renamed /KEG1/Driver/OUT+
- net /Dispenser 1/Driver/OUT- renamed /KEG1/Driver/OUT-
- net /Dispenser 1/Driver/RON renamed /KEG1/Driver/RON
- net /Dispenser 1/Driver/SW renamed /KEG1/Driver/SW
- net /Dispenser 1/Driver/VOUT renamed /KEG1/Driver/VOUT
- net /Dispenser 1/FAN renamed /KEG1/FAN
- net /Dispenser 1/VCC_FLOW renamed /KEG1/VCC_FLOW
- net /Dispenser 1/VCC_PRESS renamed /KEG1/VCC_PRESS
- net /Dispenser 1/WP renamed /KEG1/WP
- net /Dispenser 2/AP renamed /KEG2/AP
- net /Dispenser 2/Driver/BOOT renamed /KEG2/Driver/BOOT
- net /Dispenser 2/Driver/CS renamed /KEG2/Driver/CS
- net /Dispenser 2/Driver/HG renamed /KEG2/Driver/HG
- net /Dispenser 2/Driver/LG renamed /KEG2/Driver/LG
- net /Dispenser 2/Driver/OUT+ renamed /KEG2/Driver/OUT+
- net /Dispenser 2/Driver/OUT- renamed /KEG2/Driver/OUT-
- net /Dispenser 2/Driver/RON renamed /KEG2/Driver/RON
- net /Dispenser 2/Driver/SW renamed /KEG2/Driver/SW
- net /Dispenser 2/Driver/VOUT renamed /KEG2/Driver/VOUT
- net /Dispenser 2/FAN renamed /KEG2/FAN
- net /Dispenser 2/VCC_FLOW renamed /KEG2/VCC_FLOW
- net /Dispenser 2/VCC_PRESS renamed /KEG2/VCC_PRESS
- net /Dispenser 2/WP renamed /KEG2/WP
- net /MCU/BL_A renamed /MCU/UI/BL_A
- net /MCU/BL_K renamed /MCU/UI/BL_K
- net /Power/5V_EN renamed /PWR/5V_EN
- net /Power/5V_FB renamed /PWR/5V_FB
- net /Power/VR_{PRI} renamed /PWR/VR_{PRI}
- net /Power/VR_{SEC} renamed /PWR/VR_{SEC}
- net Net-(J13-Pin_2) renamed /BAT/BATT_P
- C108 pad 1: /MCU/DAC_REF -> VCC
- C63 pad 1: VCC -> /EXP/DAC_REF
- J2 pad 2: /MCU/LCD_RSTn -> /MCU/UI/LCD_RSTn
- R11 pad 1: /MCU/LCD_RSTn -> GND
- R11 pad 2: +3.3V -> /MCU/BUZZ
- R2 pad 1: /MCU/ENC_A -> GND
- R2 pad 2: Net-(R2-Pad2) -> /MCU/LCD_BL
- R3 pad 1: /MCU/ENC_B -> /MCU/LCD_BL
- R3 pad 2: Net-(R3-Pad2) -> Net-(Q1-G)
- R5 pad 1: +3.3V -> /MCU/ENC_A
- R5 pad 2: Net-(R2-Pad2) -> Net-(R5-Pad2)
- R51 pad 1: GND -> /MCU/BUZZ
- R51 pad 2: /MCU/BUZZ -> Net-(Q14-G)
- R52 pad 1: /MCU/BUZZ -> /MCU/UI/LCD_RSTn
- R52 pad 2: Net-(Q14-G) -> +3.3V
- R58 pad 1: /MCU/APEN2 -> /AP_EN_2
- R58 pad 2: Net-(U12-PWM2) -> Net-(U13-PWM2)
- R6 pad 1: +3.3V -> /MCU/ENC_B
- R6 pad 2: Net-(R3-Pad2) -> Net-(R6-Pad2)
- R60 pad 1: /AP_EN_1 -> /AP_G_1
- R77 pad 1: /AP_EN_2 -> /AP_G_2
- R8 pad 1: GND -> +3.3V
- R8 pad 2: /MCU/LCD_BL -> Net-(R5-Pad2)
- R9 pad 1: /MCU/LCD_BL -> +3.3V
- R9 pad 2: Net-(Q1-G) -> Net-(R6-Pad2)
- SW3 pad A: Net-(R2-Pad2) -> Net-(R5-Pad2)
- SW3 pad B: Net-(R3-Pad2) -> Net-(R6-Pad2)
- U12 pad 1: unconnected-(U12-EN1-Pad1) -> /~{CHG_EN}
- U12 pad 2: Net-(U12-PWM1) -> /~{CHGOK}
- U12 pad 3: GND -> /~{ACOK}
- U12 pad 4: Net-(U12-PWM2) -> GND
- U12 pad 5: /AP_EN_2 -> /~{DCIN}
- U12 pad 6: VCC -> /SCL
- U12 pad 7: /AP_EN_1 -> /SDA
- U12 pad 8: unconnected-(U12-EN2-Pad8) -> +3.3V
- U16 pad 2: /MCU/DAC_REF -> /EXP/DAC_REF
- U3 pad 4: /MCU/APEN1 -> /AP_EN_1
- U3 pad 5: /MCU/APEN2 -> /AP_EN_2
Routing:
- net /KEG2/Driver/OUT+: track 0.00 -> 23.7 mm
- net /KEG2/Driver/LG: track 0.00 -> 22.2 mm
- net /KEG1/Driver/OUT-: track 21.9 -> 6.22 mm
- net /KEG2/Driver/HG: track 0.00 -> 13.2 mm
- net VCC: track 10.3 -> 22.6 mm
- net GND: track 52.1 -> 42.2 mm, vias 11 -> 1
- net /KEG2/VCC_FLOW: track 0.00 -> 9.91 mm
- net /KEG1/Driver/OUT+: track 14.6 -> 23.7 mm
- net /KEG2/Driver/SW: track 0.00 -> 8.78 mm
- net /FAN_TACH_2: track 3.19 -> 11.5 mm
- net /KEG2/VCC_PRESS: track 0.00 -> 7.69 mm
- net /KEG2/Driver/VOUT: track 0.00 -> 7.46 mm, vias 0 -> 2
- net /KEG2/Driver/BOOT: track 0.00 -> 6.86 mm
- net /KEG2/Driver/OUT-: track 0.00 -> 6.26 mm
- net Net-(J17-Pin_2): track 0.00 -> 5.90 mm
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- added copper zone on F.Cu, net /BAT/CHG_CS+
- added copper zone on F.Cu, net /KEG1/Driver/OUT+
- added copper zone on F.Cu, net /KEG1/Driver/OUT-
- added copper zone on F.Cu, net /KEG2/Driver/OUT-
- added copper zone on F.Cu, net /KEG2/Driver/SW
- added copper zone on F.Cu, net /KEG2/FAN
- added copper zone on F.Cu, net /KEG2/WP

Commit message: layout
Parts:
- added HS1: Heatsink, portabeer:Heatsink_14x14x6mm_adhesive, B.Cu at (208.5, 105.2)
- added HS2: Heatsink, portabeer:Heatsink_14x14x6mm_adhesive, B.Cu at (234.2, 105.2)
- added HS3: Heatsink, portabeer:Heatsink_9x9x5mm_adhesive, B.Cu at (208.0, 87.5)
- JP6, JP7, JP8, JP9: moved to B.Cu
- moved C108 66.8 mm to (254.9, 107.8)
- moved R66 60.5 mm to (206.5, 57.2)
- moved R83 57.1 mm to (206.5, 55.8)
- moved R54 56.4 mm to (255.0, 99.0), turned to -90 degrees
- moved R58 53.5 mm to (253.5, 99.0), turned to -90 degrees
- moved C48 40.9 mm to (203.5, 68.8)
- moved JP4 40.9 mm to (204.0, 72.0)
- moved U10 40.9 mm to (206.5, 69.0)
- moved R45 40.7 mm to (203.7, 63.8), turned to 90 degrees
- moved R42 37.0 mm to (207.2, 65.0), turned to 90 degrees
- moved D6 36.8 mm to (201.5, 65.5), turned to 90 degrees
- moved JP5 34.7 mm to (215.2, 78.2), turned to 0 degrees
- moved R35 33.9 mm to (198.8, 64.2), turned to 180 degrees
- moved R36 33.1 mm to (198.8, 65.8), turned to 180 degrees
- moved C83 32.3 mm to (210.2, 60.2), turned to -90 degrees
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Connections:
- net Net-(F3-Pad1) renamed /BAT/VDC_UF
- J13 pad : (no net) -> VCC
Routing:
- net VCC: track 22.6 -> 71.5 mm, vias 0 -> 25
- net +3.3V: track 95.0 -> 132.2 mm
- net /BAT_NTC: track 0.00 -> 24.6 mm
- net /KEG2/Driver/OUT+: track 23.7 -> 1.35 mm
- net +5V: track 0.00 -> 19.8 mm
- net VDC: track 0.00 -> 17.1 mm
- net /KEG2/VCC_FLOW: track 9.91 -> 18.5 mm, vias 0 -> 1
- net /KEG1/VCC_FLOW: track 9.91 -> 18.5 mm, vias 0 -> 1
- net /KEG1/Driver/OUT+: track 23.7 -> 16.6 mm
- net /KEG2/VCC_PRESS: track 7.69 -> 12.8 mm, vias 0 -> 1
- net /KEG1/VCC_PRESS: track 7.69 -> 12.8 mm, vias 0 -> 1
- net Net-(J15-Pin_2): track 5.90 -> 10.6 mm
- net GND: track 42.2 -> 45.8 mm
- net Net-(J18-Pin_2): track 4.40 -> 7.97 mm
- net Net-(J16-Pin_2): track 4.40 -> 7.97 mm
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- added copper zone on F.Cu, net +BATT
- added copper zone on F.Cu, net /BAT/BATT_P
- added copper zone on F.Cu, net /BAT/BATT_PF
- added copper zone on F.Cu, net /BAT/CHG_CS-
- added copper zone on F.Cu, net /BAT/VDC_UF
- added copper zone on F.Cu, net /KEG1/AP
- added copper zone on B.Cu, net /KEG1/Driver/SW
- added copper zone on F.Cu, net /KEG2/AP
- added copper zone on B.Cu, net VCC
- added copper zone on F.Cu, net VDC

Commit message: working
Parts:
- removed C16: 100n, Capacitor_SMD:C_0603_1608Metric
- removed M3, M6: Water pump, portabeer:Molex_KK-254_1x02_P2.54mm_Horizontal
- removed M7, M8: Fan_4pin, portabeer:Molex_KK-254_1x03_P2.54mm_Horizontal
- added J19: FAN, Connector_Molex:Molex_KK-254_AE-6410-03A_1x03_P2.54mm_Vertical, F.Cu at (271.5, 90.5)
- added J20: FAN, Connector_Molex:Molex_KK-254_AE-6410-03A_1x03_P2.54mm_Vertical, F.Cu at (271.5, 81.8)
- added J21: WATER PUMP, Connector_Molex:Molex_KK-254_AE-6410-02A_1x02_P2.54mm_Vertical, F.Cu at (271.5, 103.8)
- added J22: WATER PUMP, Connector_Molex:Molex_KK-254_AE-6410-02A_1x02_P2.54mm_Vertical, F.Cu at (271.5, 96.8)
- added R68: 0, Resistor_SMD:R_0603_1608Metric, F.Cu at (203.2, 88.0)
- moved U17 5.49 mm to (237.0, 84.8), turned to 180 degrees
- moved C63 5.11 mm to (237.2, 82.2), turned to 180 degrees
- moved C86 5.10 mm to (237.2, 87.2), turned to 180 degrees
- moved U16 3.04 mm to (240.8, 84.0)
- moved R59 2.36 mm to (237.2, 80.8)
- moved R41 1.46 mm to (195.2, 98.8)
- moved C96 1.25 mm to (219.2, 99.2)
- moved R43 1.00 mm to (203.2, 89.5)
- moved R44 1.00 mm to (203.2, 91.0)
- moved R47 1.00 mm to (203.3, 92.5)
Connections:
- J13 pad : VCC -> (no net)
- U11 pad 2: /BAT_NTC -> Net-(U11-NTC)
Routing:
- net VCC: track 71.5 -> 82.9 mm, vias 25 -> 89
- net Net-(U11-NTC): track 0.00 -> 2.43 mm
- net /FAN_TACH_2: track 10.6 -> 12.1 mm
- net /FAN_TACH_1: track 9.23 -> 10.7 mm
- net /BAT/BATT_PF: track 3.95 -> 5.38 mm, vias 0 -> 2
- net GND: track 45.8 -> 46.6 mm, vias 1 -> 32
- net /BAT_NTC: track 24.6 -> 23.9 mm
Other:
- board text added: "0.5mm via hole -> ~1mOhm/via"
- board text added: "BOOT"
- board text added: "RESET"

Commit message: partial routing
Parts:
- removed C72, C87: 1u, Capacitor_SMD:C_0603_1608Metric
- removed C80: C, Capacitor_SMD:C_0603_1608Metric
- removed C84: 10u, Capacitor_SMD:C_1206_3216Metric
- removed C85: 1n, Capacitor_SMD:C_0603_1608Metric
- removed J18: Conn_01x03, Connector_JST:JST_XH_B3B-XH-A_1x03_P2.50mm_Vertical
- removed M4: Air pump, Connector_Phoenix_MC:PhoenixContact_MC_1,5_2-G-3.81_1x02_P3.81mm_Horizontal
- removed Q9: SiS454DN, portabeer:Vishay_PowerPAK_1212-8_Single
- removed R77: 10, Resistor_SMD:R_0603_1608Metric
- removed R78: 1k, Resistor_SMD:R_0603_1608Metric
- removed R79: 1.96k, Resistor_SMD:R_0603_1608Metric
- removed TP1: IO20, TestPoint:TestPoint_THTPad_1.0x1.0mm_Drill0.5mm
- removed U13: GBI7254MMAR, Package_SO:MSOP-8-1EP_3x3mm_P0.65mm_EP1.95x2.15mm
- added C54: 10u, Capacitor_SMD:C_1206_3216Metric, F.Cu at (259.0, 115.5)
- added C60: 1u, Capacitor_SMD:C_0603_1608Metric, F.Cu at (257.0, 115.5)
- added C67: 1n, Capacitor_SMD:C_0603_1608Metric, F.Cu at (262.8, 74.8)
- added C68: 100n, Capacitor_SMD:C_0603_1608Metric, F.Cu at (221.2, 34.5)
- added JP10: SolderJumper_2_Open, Jumper:SolderJumper-2_P1.3mm_Open_RoundedPad1.0x1.5mm, B.Cu at (263.5, 85.2)
- added JP11: SolderJumper_2_Open, Jumper:SolderJumper-2_P1.3mm_Open_RoundedPad1.0x1.5mm, B.Cu at (263.5, 79.2)
- added R69: 1k, Resistor_SMD:R_0603_1608Metric, F.Cu at (184.8, 37.2)
- added U4: COS1416, Package_TO_SOT_SMD:SOT-23-5, F.Cu at (252.5, 106.2)
- C57: footprint Capacitor_THT:CP_Radial_D8.0mm_P3.50mm -> Capacitor_THT:CP_Radial_D6.3mm_P2.50mm
- C69: value 10u -> 100n; footprint Capacitor_SMD:C_1206_3216Metric -> Capacitor_SMD:C_0603_1608Metric
- C70: value 1n -> 100n
- D1: value LED -> LED_GREEN
- D12: value PMEG3030EP -> LED_YELLOW; footprint Diode_SMD:D_SOD-128 -> LED_SMD:LED_0603_1608Metric
- J4: value I2C expansion -> Conn_01x08; footprint Connector_PinHeader_2.54mm:PinHeader_1x05_P2.54mm_Vertical -> Connector_PinHeader_2.54mm:PinHeader_1x08_P2.54mm_Vertical
- JP9: value SolderJumper_3_Open -> SolderJumper_2_Open; footprint Jumper:SolderJumper-3_P1.3mm_Open_RoundedPad1.0x1.5mm -> Jumper:SolderJumper-2_P1.3mm_Open_RoundedPad1.0x1.5mm
- R58: value 100 -> 10k
- moved D12 113.4 mm to (184.8, 34.2), turned to -90 degrees
- moved C69 106.4 mm to (193.8, 31.2), turned to -90 degrees
- moved JP9 47.7 mm to (263.5, 92.8), turned to 90 degrees
- moved R17 37.4 mm to (201.2, 65.8)
- moved R16 36.2 mm to (199.8, 65.8)
- moved Q3 33.0 mm to (214.2, 70.2), turned to 90 degrees
- moved C47 29.4 mm to (214.2, 67.5), turned to 180 degrees
- moved C70 28.7 mm to (227.2, 33.2), turned to 180 degrees
- moved J16 28.2 mm to (268.0, 77.8)
- moved J17 28.2 mm to (268.0, 84.0)
- moved J15 28.2 mm to (268.0, 90.2)
- moved R42 27.8 mm to (186.8, 83.8), turned to 180 degrees
- moved C48 27.0 mm to (186.5, 89.8), turned to 0 degrees
- moved C62 26.7 mm to (264.2, 88.2)
- moved C64 26.7 mm to (262.8, 88.2)
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Connections:
- net /KEG1/AP renamed /EXP/AP
- net /KEG1/VCC_PRESS renamed /EXP/VCC_PRESS
- net Net-(D4-K) renamed /BAT/VDC_SCAL
- C69 pad 1: VCC -> +5V
- C70 pad 1: /PRESS_1 -> +3.3V
- D12 pad 1: VCC -> GND
- D12 pad 2: /KEG2/AP -> Net-(D12-A)
- D2 pad 1: +BATT -> VDC
- D2 pad 2: VDC -> +BATT
- J4 pad 4: +3.3V -> /IO29
- J4 pad 5: +5V -> /IO25
- JP9 pad 1: +3.3V -> GND
- JP9 pad 2: /KEG2/VCC_PRESS -> Net-(JP9-B)
- R54 pad 1: /AP_EN_1 -> /AP_EN
- R57 pad 1: GND -> Net-(JP9-B)
- R58 pad 1: /AP_EN_2 -> /AP_EN
- R58 pad 2: Net-(U13-PWM2) -> GND
- R60 pad 1: /AP_G_1 -> Net-(U4-OUT)
- R61 pad 1: /PRESS_1 -> /PRESS
- R62 pad 1: GND -> Net-(JP11-B)
- R62 pad 2: /PRESS_1 -> /PRESS
- R74 pad 1: GND -> Net-(JP10-B)
- U3 pad 31: /MCU/LCD_MISO -> /IO20
- U3 pad 36: /MCU/LCD_BL -> /MCU/BUZZ
- U3 pad 37: /MCU/BUZZ -> /IO25
- U3 pad 4: /AP_EN_1 -> /AP_EN
- U3 pad 40: /PRESS_1 -> /PRESS
- U3 pad 41: /PRESS_2 -> /IO29
- U3 pad 5: /AP_EN_2 -> /MCU/LCD_BL
Routing:
- net /SDA: track 1.40 -> 139.3 mm, vias 0 -> 8
- net /SCL: track 1.40 -> 136.9 mm, vias 0 -> 5
- net /TE_EN_1: track 4.99 -> 121.6 mm
- net /WP_EN_1: track 1.50 -> 114.6 mm
- net /WP_EN_2: track 1.50 -> 109.0 mm
- net /PRESS: track 0.00 -> 105.1 mm
- net /BAT_NTC: track 23.9 -> 124.6 mm, vias 0 -> 8
- net /FAN_EN_1: track 1.50 -> 99.8 mm
- net /AP_EN: track 0.00 -> 95.6 mm
- net /TE_EN_2: track 3.74 -> 99.1 mm
- net /FAN_EN_2: track 1.50 -> 92.7 mm
- net /FAN_TACH_1: track 10.7 -> 92.7 mm, vias 0 -> 1
- net +BATT: track 4.55 -> 81.0 mm, vias 0 -> 2
- net /IO29: track 0.00 -> 73.9 mm
- net /FAN_TACH_2: track 12.1 -> 84.7 mm
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- added copper zone on F.Cu, net +1V1
- added copper zone on F.Cu, net +3.3V
- added copper zone on F.Cu, net +3.3VA
- removed copper zone on F.Cu, net /KEG2/AP
Other:
- outline, holes or cut-outs redrawn
- board text added: "INFO"
- board text added: "PWR"
