File: portabeer_pcb/mcu.kicad_sch (KiCad schematic)
At the start: 65 parts, among them J1 USB_B_Micro, J2 GMG12864-06D, J3 Conn_01x03, J4 I2C expansion, Q1 AO3400A, SW1 RESET, SW2 BOOTSEL, SW3 RotaryEncoder_Switch_MP, U1 USBLC6-2SC6, U12 GBI7254MMAR, U16 MCP47FEB12, U18 REF3025, U2 W25Q128JVS, U3 RP2040, U4 PCA9536DP, Y1 Crystal_GND24

Commit message: electronics diagram and schematic
Parts:
- removed C1, C108, C16, C2, C63, C83, C86: 100n, Capacitor_SMD:C_0603_1608Metric, symbol Device:C
- removed H1, H2: MountingHole, MountingHole:MountingHole_2.7mm_M2.5, symbol Mechanical:MountingHole
- removed J2: GMG12864-06D, portabeer:GMG12864-06D, symbol Connector_Generic:Conn_01x13
- removed J4: I2C expansion, Connector_PinHeader_2.54mm:PinHeader_1x05_P2.54mm_Vertical, symbol Connector_Generic:Conn_01x05
- removed Q1: AO3400A, Package_TO_SOT_SMD:SOT-23, symbol Transistor_FET:AO3400A
- removed R10: R, Resistor_SMD:R_0805_2012Metric, symbol Device:R
- removed R11, R8: 10k, Resistor_SMD:R_0603_1608Metric, symbol Device:R
- removed R2, R3: 10Rx, Resistor_SMD:R_0603_1608Metric, symbol Device:R
- removed R5, R6: Rx, Resistor_SMD:R_0603_1608Metric, symbol Device:R
- removed R58, R75: 100, Resistor_SMD:R_0603_1608Metric, symbol Device:R
- removed R9: 10, Resistor_SMD:R_0603_1608Metric, symbol Device:R
- removed R99: 1k, Resistor_SMD:R_0603_1608Metric, symbol Device:R
- removed SW3: RotaryEncoder_Switch_MP, Rotary_Encoder:RotaryEncoder_Alps_EC11E-Switch_Vertical_H20mm, symbol Device:RotaryEncoder_Switch_MP
- removed U12: GBI7254MMAR, Package_SO:MSOP-8-1EP_3x3mm_P0.65mm_EP1.95x2.15mm, symbol Driver_FET:PM8834M
- removed U16: MCP47FEB12, Package_SO:TSSOP-8_4.4x3mm_P0.65mm, symbol portabeer:MCP47FEB12
- removed U18: REF3025, Package_TO_SOT_SMD:SOT-23, symbol Reference_Voltage:REF3025
- removed U4: PCA9536DP, Package_SO:TSSOP-8_3x3mm_P0.65mm, symbol Interface_Expansion:PCA9536DP
Connections:
- net APEN1 is gone; now on net AP_EN_1: U3.4 (GPIO2)
- net APEN2 is gone; now on net AP_EN_2: U3.5 (GPIO3)
- net +3.3V: now also R15.2
- net GPIO25 renamed BUZZ
- net BUZZ: no longer R15.2
- no-connect marks 4 -> 0
Other:
- added sheet UI (ui.kicad_sch)
- company: Luca Anastasio -> ©2024 Luca Anastasio
- title: (none) -> Beerpak
- moved on the sheet: R1, R4, R7, SW1, SW2, U2

Commit message: added 3d models, started layout
Parts:
- J1: footprint Connector_USB:USB_Micro-B_Amphenol_10118193-0001LF_Horizontal -> portabeer:USB_Micro-B_Amphenol_10118193-0001LF_Horizontal
- U2: footprint Package_SO:SOIC-8_5.23x5.23mm_P1.27mm -> portabeer:SOIC-8_5.23x5.23mm_P1.27mm
Changed lines of the file:
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@@
 			)
 		)
-		(property "Footprint" "Connector_USB:USB_Micro-B_Amphenol_10118193-0001LF_Horizontal"
+		(property "Footprint" "portabeer:USB_Micro-B_Amphenol_10118193-0001LF_Horizontal"
 			(at 27.94 74.93 0)
 			(effects
@@
 			)
 		)
-		(property "Footprint" "Package_SO:SOIC-8_5.23x5.23mm_P1.27mm"
+		(property "Footprint" "portabeer:SOIC-8_5.23x5.23mm_P1.27mm"
 			(at 77.47 163.83 0)
 			(effects

Commit message: partial routing
Parts:
- removed TP1: IO20, TestPoint:TestPoint_THTPad_1.0x1.0mm_Drill0.5mm, symbol Connector:TestPoint
- added D12: LED_YELLOW, LED_SMD:LED_0603_1608Metric, symbol Device:LED
- added R69: 1k, Resistor_SMD:R_0603_1608Metric, symbol Device:R
- D1: value LED -> LED_GREEN
Connections:
- net AP_EN_2 is gone; now on net LCD_BL: U3.5 (GPIO3)
- net BUZZ: now also U3.36 (GPIO24); no longer U3.37 (GPIO25)
- net GND: now also D12.1 (K)
- net LCD_BL: no longer U3.36 (GPIO24)
- net AP_EN_1 renamed AP_EN
- net LCD_MISO renamed IO20
- net PRESS_1 renamed PRESS
- net PRESS_2 renamed IO29
- new net: D12.2 (A), R69.1
- new net IO25: R69.2, U3.37 (GPIO25)
Other:
- note added: "(LCD_MISO)"
- note added: "(LED)"

Commit message: layout
Parts:
- added R70: 10k, Resistor_SMD:R_0603_1608Metric, symbol Device:R
- added TH1: Thermistor_NTC, Resistor_SMD:R_0603_1608Metric_Pad0.98x0.95mm_HandSolder, symbol Device:Thermistor_NTC
Connections:
- net +3.3V: now also R70.2
- net GND: now also TH1.2
- net IO20 renamed PCB_FAN
- net IO29 renamed PCB_NTC
- net PCB_NTC: now also R70.1, TH1.1
