File: portabeer_pcb/portabeer_pcb.kicad_sch (KiCad schematic)
At the start: 4 parts

Commit message: electronics diagram and schematic
Other:
- sheet Battery renamed BAT
- sheet Dispenser 1 renamed KEG1
- sheet Dispenser 2 renamed KEG2
- sheet Power renamed PWR
- added sheet EXP (exp.kicad_sch)
- sheet MCU ports: added none; removed TE_REF_1, TE_REF_2, ~{ACOK}, ~{CHGOK}, ~{CHG_EN}, ~{DCIN}
- company: (none) -> ©2024 Luca Anastasio
- title: (none) -> Beerpak

Commit message: partial routing
Other:
- sheet EXP ports: added AP_EN, IO[0..29], PRESS; removed AP_EN_1, AP_EN_2, AP_G_1, AP_G_2
- sheet KEG1 ports: added none; removed AP_EN, PRESS
- sheet KEG2 ports: added none; removed AP_EN, PRESS
- sheet MCU ports: added AP_EN, IO[0..29], PRESS; removed AP_EN_1, AP_EN_2, PRESS_1, PRESS_2
- note added: "DAC, I2C expander and air pump"

Commit message: layout
Parts:
- added H10, H11, H12, H9: MountingHole_Pad, MountingHole:MountingHole_3.2mm_M3_Pad, symbol Mechanical:MountingHole_Pad
Connections:
- new net GND: H10.1, H11.1, H12.1, H9.1
Other:
- sheet EXP ports: added FAN_EN; removed none
- sheet MCU ports: added PCB_FAN; removed none
