File: portabeer_pcb/ui.kicad_sch (KiCad schematic)
At the start: 20 parts, among them J2 GMG12864-06D, Q1 AO3400A, Q14 AO3400A, SW3 RotaryEncoder_Switch_MP

Commit message: added 3d models, started layout
Parts:
- SW3: footprint Rotary_Encoder:RotaryEncoder_Alps_EC11E-Switch_Vertical_H20mm -> portabeer:RotaryEncoder_Alps_EC11E-Switch_Vertical_H20mm
Changed lines of the file:
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@@
 			)
 		)
-		(property "Footprint" "Rotary_Encoder:RotaryEncoder_Alps_EC11E-Switch_Vertical_H20mm"
+		(property "Footprint" "portabeer:RotaryEncoder_Alps_EC11E-Switch_Vertical_H20mm"
 			(at 201.93 54.356 0)
 			(effects

Commit message: partial routing
Parts:
- added C68, C69, C70: 100n, Capacitor_SMD:C_0603_1608Metric, symbol Device:C
Connections:
- net +3.3V: now also C70.1
- net +5V: now also C68.1, C69.1
- net GND: now also C68.2, C69.2, C70.2

Commit message: layout
Parts:
- added H7, H8: MountingHole_Pad, MountingHole:MountingHole_2.7mm_M2.5_Pad, symbol Mechanical:MountingHole_Pad
Connections:
- net GND: now also H7.1, H8.1
